File: dev_board.kicad_pcb (KiCad board)
At the start: 2 copper layers, 64 parts, among them J1 USB_B_Micro, J2 ARJ-169, J3 Conn_02x10_Odd_Even, J4 Conn_02x10_Odd_Even, SW1 SW_Push, U1 LTC3604_UD, U2 KSZ8081RND, U3 93LCxxB, U4 FT232H, U5 STM32F107RCTx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

Commit message: redirected 3D models for custom footprints on PCB
Parts:
- U1: footprint Housings_DFN_QFN:QFN-16-1EP_3x3mm_Pitch0.5mm_ThermalVias -> Exodus_Packages:QFN-16-1EP_3x3mm_P0.5mm
- moved U1 0.06 mm to (99.6, 87.6)
Connections:
- net Net-(U2-Pad7) renamed /ethernet_phy_ksz8081/OSC_OUT
- R10 pad 1: Net-(R10-Pad1) -> /stm32f107/ETH_RMII_CRS_DV
- R11 pad 1: Net-(R11-Pad1) -> /ethernet_phy_ksz8081/RMII_RXER
- R6 pad 2: Net-(R6-Pad2) -> /stm32f107/ETH_RMII_MDIO
- R8 pad 2: Net-(R8-Pad2) -> /ethernet_phy_ksz8081/INTRP
