File: dev_board.kicad_pcb (KiCad board)
At the start: 2 copper layers, 76.3 x 43.7 mm, 63 parts, among them J1 USB_B_Micro, J2 ARJ-169, J3 Conn_02x10_Odd_Even, J4 Conn_02x10_Odd_Even, SW1 SW_Push, U1 LTC3604_UD, U2 KSZ8081RND, U3 93LCxxB, U4 FT232H, U5 STM32F107RCTx, Y1 Crystal, Y2 Crystal

Commit message: pcb updates or something
Parts:
- removed R12, R7: 1M DNP, Resistors_SMD:R_0603
- removed R9: 10K DNP, Resistors_SMD:R_0603
- added D1: LED, LEDs:LED_0603, F.Cu at (119.9, 84.1)
- added R17: R, Resistors_SMD:R_0603, F.Cu at (119.9, 87.4)
- added R18: R, Resistors_SMD:R_0603, F.Cu at (72.6, 105.4)
- added R19: R, Resistors_SMD:R_0603, F.Cu at (85.6, 102.5)
- Y1, Y2: value Crystal -> Crystal_GND24; footprint Crystals:Crystal_SMD_0603-4pin_6.0x3.5mm_HandSoldering -> Crystals:Crystal_SMD_3225-4pin_3.2x2.5mm
- moved J3 77.2 mm to (122.9, 83.7), turned to 0 degrees
- moved C16 50.2 mm to (41.3, 78.8)
- moved C15 49.9 mm to (36.4, 83.1)
- moved R10 46.0 mm to (44.0, 83.4)
- moved R11 43.8 mm to (49.3, 82.9)
- moved R8 42.3 mm to (49.8, 85.9)
- moved R1 41.6 mm to (54.7, 113.2), turned to 180 degrees
- moved SW1 41.1 mm to (61.7, 113.3), turned to 270 degrees
- moved C3 41.0 mm to (54.9, 114.6), turned to 0 degrees
- moved J1 37.0 mm to (126.0, 114.0), turned to 90 degrees
- moved C10 35.9 mm to (88.5, 92.1), turned to 90 degrees
- moved L1 30.9 mm to (93.1, 92.6), turned to 270 degrees
- moved R6 30.1 mm to (53.5, 84.3)
- moved Y1 28.4 mm to (109.6, 99.4), turned to 180 degrees
- moved C9 25.1 mm to (97.3, 91.2), turned to 180 degrees
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Connections:
- net /ethernet_phy_ksz8081/OSC_OUT renamed Net-(U2-Pad7)
- C32 pad 1: /stm32f107/OSC2 -> GND
- C32 pad 2: GND -> /stm32f107/OSC2
- J1 pad 1: +5V -> Net-(J1-Pad1)
- J2 pad 13: Net-(J2-Pad13) -> GND
- J2 pad 15: Net-(J2-Pad15) -> GND
- R10 pad 1: /stm32f107/ETH_RMII_CRS_DV -> Net-(R10-Pad1)
- R11 pad 1: /ethernet_phy_ksz8081/RMII_RXER -> Net-(R11-Pad1)
- R6 pad 2: /stm32f107/ETH_RMII_MDIO -> Net-(R6-Pad2)
- R8 pad 2: /ethernet_phy_ksz8081/INTRP -> Net-(R8-Pad2)
- Y1 pad 2: Net-(C20-Pad1) -> GND
- Y1 pad 3: (no net) -> Net-(C20-Pad1)
- Y1 pad 4: (no net) -> GND
- Y2 pad 2: /stm32f107/OSC2 -> GND
- Y2 pad 3: (no net) -> /stm32f107/OSC2
- Y2 pad 4: (no net) -> GND
Routing:
- net /stm32f107/MCO: track 0.00 -> 32.9 mm
- net /NRST: track 30.0 -> 0.00 mm
- net /stm32f107/ETH_RMII_MDC: track 3.47 -> 30.0 mm, vias 0 -> 2
- net /stm32f107/ETH_RMII_MDIO: track 4.04 -> 29.0 mm, vias 0 -> 2
- net /stm32f107/OTG_FS_P: track 36.4 -> 60.6 mm
- net /stm32f107/OTG_FS_N: track 35.8 -> 59.1 mm
- net +5V: track 34.4 -> 12.1 mm
- net +3V3: track 30.1 -> 10.3 mm
- net /stm32f107/ETH_RMII_RXD1: track 0.00 -> 17.3 mm
- net /stm32f107/ETH_RMII_RXD0: track 0.00 -> 16.0 mm
- net /ethernet_phy_ksz8081/INTRP: track 3.60 -> 18.8 mm, vias 0 -> 2
- net /TDO: track 14.2 -> 0.00 mm
- net /TMS: track 12.3 -> 0.00 mm
- net /stm32f107/ETH_RMII_CRS_DV: track 2.81 -> 14.2 mm
- net /TDI: track 11.2 -> 0.00 mm
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
Commit message: revised ethernet layout
Parts:
- removed R8: 1K, Resistors_SMD:R_0603
- R10, R11, R6: footprint Resistors_SMD:R_0603 -> Resistor_SMD:R_0603_1608Metric
- Y1: value Crystal_GND24 -> Crystal; footprint Crystals:Crystal_SMD_3225-4pin_3.2x2.5mm -> Crystal:Crystal_HC49-U_Vertical
- moved C16 43.6 mm to (71.6, 110.1), turned to 180 degrees
- moved C15 43.5 mm to (71.6, 108.6), turned to 180 degrees
- moved R6 40.3 mm to (90.2, 100.8), turned to 270 degrees
- moved R10 39.5 mm to (71.6, 111.6), turned to 180 degrees
- moved R11 37.8 mm to (71.6, 113.4), turned to 180 degrees
- moved R1 12.5 mm to (66.5, 117.1)
- moved C3 11.7 mm to (66.5, 115.6)
- moved R13 11.0 mm to (82.8, 110.7)
- moved R18 9.33 mm to (77.0, 113.7), turned to 90 degrees
- moved L2 7.88 mm to (80.5, 113.2), turned to 0 degrees
- moved C19 7.14 mm to (103.9, 93.6), turned to 180 degrees
- moved C12 7.14 mm to (80.5, 116.2)
- moved C14 7.01 mm to (80.5, 114.7)
- moved Y1 6.70 mm to (108.7, 92.7), turned to 270 degrees
- moved C11 6.40 mm to (80.5, 111.6), turned to 0 degrees
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Connections:
- net Net-(U2-Pad7) renamed /ethernet_phy_ksz8081/OSC_OUT
- R10 pad 1: Net-(R10-Pad1) -> /stm32f107/ETH_RMII_CRS_DV
- R11 pad 1: Net-(R11-Pad1) -> /ethernet_phy_ksz8081/RMII_RXER
- R6 pad 2: Net-(R6-Pad2) -> /stm32f107/ETH_RMII_MDIO
- Y1 pad 2: GND -> Net-(C20-Pad1)
Routing:
- net /stm32f107/OTG_FS_P: track 60.6 -> 0.00 mm
- net /stm32f107/OTG_FS_N: track 59.1 -> 0.00 mm
- net Net-(J2-Pad14): track 1.75 -> 16.7 mm, vias 0 -> 1
- net /stm32f107/ETH_RMII_CRS_DV: track 14.2 -> 28.1 mm
- net GND: track 72.4 -> 85.1 mm, vias 54 -> 56
- net /NRST: track 0.00 -> 9.70 mm
- net /stm32f107/ETH_RMII_TX_EN: track 11.2 -> 19.1 mm
- net Net-(C19-Pad1): track 8.44 -> 16.3 mm
- net /ethernet_phy_ksz8081/INTRP: track 18.8 -> 26.0 mm, vias 2 -> 0
- net /ethernet_phy_ksz8081/PHY_REF_RES: track 3.16 -> 9.58 mm, vias 0 -> 2
- net /stm32f107/ETH_RMII_TXD0: track 14.4 -> 20.6 mm, vias 2 -> 0
- net /stm32f107/ETH_RMII_TXD1: track 16.0 -> 22.1 mm, vias 2 -> 0
- net /stm32f107/MCO: track 32.9 -> 27.0 mm
- net /RX_N: track 11.2 -> 15.7 mm, vias 0 -> 1
- net /ethernet_phy_ksz8081/RMII_RXER: track 0.00 -> 4.44 mm
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