File: power_supply.sch (KiCad schematic (older format))
At the start: 12 parts, among them U100 LT8609

Commit message: added footprints for power components. Updated netlist.
Parts:
- C100, C101, C102, C103, C104: footprint (none) -> Capacitors_SMD:C_0603
- C105: value C_Small -> 22uF; footprint (none) -> Capacitors_SMD:C_0603
- L100: footprint (none) -> Inductors_SMD:L_Vishay_IHLP-2020
- R100, R101, R102, R103: footprint (none) -> Resistors_SMD:R_0603
Changed lines of the file:
@@
 F 0 "C100" H 4710 3220 50  0000 L CNN
 F 1 "4.7uF" H 4710 3070 50  0000 L CNN
-F 2 "" H 4700 3150 50  0001 C CNN
+F 2 "Capacitors_SMD:C_0603" H 4700 3150 50  0001 C CNN
 F 3 "" H 4700 3150 50  0001 C CNN
 	1    4700 3150
@@
 F 0 "C101" H 4400 3700 50  0000 L CNN
 F 1 "1uF" H 4450 3500 50  0000 L CNN
-F 2 "" H 4600 3600 50  0001 C CNN
+F 2 "Capacitors_SMD:C_0603" H 4600 3600 50  0001 C CNN
 F 3 "" H 4600 3600 50  0001 C CNN
 	1    4600 3600
@@
 F 0 "C102" H 4650 3800 50  0000 L CNN
 F 1 "10nF" H 4650 3650 50  0000 L CNN
-F 2 "" H 4750 3700 50  0001 C CNN
+F 2 "Capacitors_SMD:C_0603" H 4750 3700 50  0001 C CNN
 F 3 "" H 4750 3700 50  0001 C CNN
 	1    4750 3700
@@
 F 0 "R100" H 4930 3820 50  0000 L CNN
 F 1 "18.2k" H 4930 3760 50  0000 L CNN
-F 2 "" H 4900 3800 50  0001 C CNN
+F 2 "Resistors_SMD:R_0603" H 4900 3800 50  0001 C CNN
 F 3 "" H 4900 3800 50  0001 C CNN
 	1    4900 3800
@@
 F 0 "R102" H 6080 3770 50  0000 L CNN
 F 1 "309k" H 6080 3710 50  0000 L CNN
-F 2 "" H 6050 3750 50  0001 C CNN
+F 2 "Resistors_SMD:R_0603" H 6050 3750 50  0001 C CNN
 F 3 "" H 6050 3750 50  0001 C CNN
 	1    6050 3750
@@
 F 0 "R103" H 6430 3770 50  0000 L CNN
 F 1 "1M" H 6430 3710 50  0000 L CNN
-F 2 "" H 6400 3750 50  0001 C CNN
+F 2 "Resistors_SMD:R_0603" H 6400 3750 50  0001 C CNN
 F 3 "" H 6400 3750 50  0001 C CNN
 	1    6400 3750
@@
 F 0 "C104" H 6410 3670 50  0000 L CNN
 F 1 "10pF" H 6410 3520 50  0000 L CNN
-F 2 "" H 6400 3600 50  0001 C CNN
+F 2 "Capacitors_SMD:C_0603" H 6400 3600 50  0001 C CNN
 F 3 "" H 6400 3600 50  0001 C CNN
 	1    6400 3600
@@
 P 6700 3800
 F 0 "C105" H 6710 3870 50  0000 L CNN
-F 1 "C_Small" H 6710 3720 50  0000 L CNN
-F 2 "" H 6700 3800 50  0001 C CNN
+F 1 "22uF" H 6710 3720 50  0000 L CNN
+F 2 "Capacitors_SMD:C_0603" H 6700 3800 50  0001 C CNN
 F 3 "" H 6700 3800 50  0001 C CNN
 	1    6700 3800
@@
 F 0 "L100" H 6450 3250 50  0000 L CNN
 F 1 "2.2uH" H 6430 3160 50  0000 L CNN
-F 2 "" H 6400 3200 50  0001 C CNN
+F 2 "Inductors_SMD:L_Vishay_IHLP-2020" H 6400 3200 50  0001 C CNN
 F 3 "" H 6400 3200 50  0001 C CNN
 	1    6400 3200
@@
 F 0 "C103" H 6160 3070 50  0000 L CNN
 F 1 "0.1uF" H 6160 2920 50  0000 L CNN
-F 2 "" H 6150 3000 50  0001 C CNN
+F 2 "Capacitors_SMD:C_0603" H 6150 3000 50  0001 C CNN
 F 3 "" H 6150 3000 50  0001 C CNN
 	1    6150 3000
@@
 F 0 "R101" H 6630 3370 50  0000 L CNN
 F 1 "100k" H 6630 3310 50  0000 L CNN
-F 2 "" H 6600 3350 50  0001 C CNN
+F 2 "Resistors_SMD:R_0603" H 6600 3350 50  0001 C CNN
 F 3 "" H 6600 3350 50  0001 C CNN
 	1    6600 3350

Commit message: Updating project to kicad 5. Added USB ports.
Parts:
- removed U100: LT8609, Housings_SSOP:MSOP-10-1EP_3x3mm_Pitch0.5mm, symbol LT8609
- added U2: LT8609, Housings_SSOP:MSOP-10-1EP_3x3mm_Pitch0.5mm, symbol lt8609:LT8609
- C1: renamed from C101; symbol C_Small -> Device:C_Small
- C2: renamed from C100; symbol C_Small -> Device:C_Small
- C3: renamed from C102; symbol C_Small -> Device:C_Small
- C4: renamed from C103; symbol C_Small -> Device:C_Small
- C5: renamed from C104; symbol C_Small -> Device:C_Small
- C6: renamed from C105; symbol C_Small -> Device:C_Small
- L1: renamed from L100; symbol L_Small -> Device:L_Small
- R1: renamed from R100; symbol R_Small -> Device:R_Small
- R2: renamed from R102; symbol R_Small -> Device:R_Small
- R3: renamed from R103; symbol R_Small -> Device:R_Small
- R4: renamed from R101; symbol R_Small -> Device:R_Small
Connections:
- wire segments 33 -> 47
Changed lines of the file:
@@
-EESchema Schematic File Version 2
-LIBS:power
-LIBS:device
-LIBS:switches
-LIBS:relays
-LIBS:motors
-LIBS:transistors
-LIBS:conn
-LIBS:linear
-LIBS:regul
-LIBS:74xx
-LIBS:cmos4000
-LIBS:adc-dac
-LIBS:memory
-LIBS:xilinx
-LIBS:microcontrollers
-LIBS:dsp
-LIBS:microchip
-LIBS:analog_switches
-LIBS:motorola
-LIBS:texas
-LIBS:intel
-LIBS:audio
-LIBS:interface
-LIBS:digital-audio
-LIBS:philips
-LIBS:display
-LIBS:cypress
-LIBS:siliconi
-LIBS:opto
-LIBS:atmel
-LIBS:contrib
-LIBS:valves
-LIBS:stm32f107xx
-LIBS:lt8609
-LIBS:dev-board-stm32f107-cache
-EELAYER 25 0
+EESchema Schematic File Version 4
+LIBS:dev_board-cache
+EELAYER 26 0
 EELAYER END
 $Descr A4 11693 8268
 encoding utf-8
-Sheet 2 2
+Sheet 2 5
 Title ""
 Date ""
@@
 $EndDescr
 $Comp
-L LT8609 U100
-U 1 1 5B330245
-P 5500 3350
-F 0 "U100" H 5700 2900 60  0000 C CNN
-F 1 "LT8609" H 5500 3800 60  0000 C CNN
-F 2 "Housings_SSOP:MSOP-10-1EP_3x3mm_Pitch0.5mm" H 5500 3800 60  0001 C CNN
-F 3 "" H 5500 3800 60  0001 C CNN
-	1    5500 3350
-	1    0    0    -1
-$EndComp
-$Comp
-L C_Small C100
+L Device:C_Small C2
 U 1 1 5B3303D0
 P 4700 3150
-F 0 "C100" H 4710 3220 50  0000 L CNN
+F 0 "C2" H 4710 3220 50  0000 L CNN
 F 1 "4.7uF" H 4710 3070 50  0000 L CNN
 F 2 "Capacitors_SMD:C_0603" H 4700 3150 50  0001 C CNN
@@
 $EndComp
 $Comp
-L GND #PWR?
+L power:GND #PWR0101
 U 1 1 5B33040E
 P 4700 3250
-F 0 "#PWR?" H 4700 3000 50  0001 C CNN
+F 0 "#PWR0101" H 4700 3000 50  0001 C CNN
 F 1 "GND" H 4700 3100 50  0000 C CNN
 F 2 "" H 4700 3250 50  0001 C CNN
@@
 $EndComp
 $Comp
-L C_Small C101
+L Device:C_Small C1
 U 1 1 5B330498
 P 4600 3600
-F 0 "C101" H 4400 3700 50  0000 L CNN
+F 0 "C1" H 4400 3700 50  0000 L CNN
 F 1 "1uF" H 4450 3500 50  0000 L CNN
 F 2 "Capacitors_SMD:C_0603" H 4600 3600 50  0001 C CNN
@@
 $EndComp
 $Comp
-L C_Small C102
+L Device:C_Small C3
 U 1 1 5B3304FE
 P 4750 3700
-F 0 "C102" H 4650 3800 50  0000 L CNN
+F 0 "C3" H 4650 3800 50  0000 L CNN
 F 1 "10nF" H 4650 3650 50  0000 L CNN
 F 2 "Capacitors_SMD:C_0603" H 4750 3700 50  0001 C CNN
@@
 $EndComp
 $Comp
-L R_Small R100
+L Device:R_Small R1
 U 1 1 5B330539
 P 4900 3800
-F 0 "R100" H 4930 3820 50  0000 L CNN
+F 0 "R1" H 4930 3820 50  0000 L CNN
 F 1 "18.2k" H 4930 3760 50  0000 L CNN
 F 2 "Resistors_SMD:R_0603" H 4900 3800 50  0001 C CNN
@@
 $EndComp
 $Comp
-L GND #PWR?
+L power:GND #PWR0102
 U 1 1 5B330A26
 P 5500 4000
-F 0 "#PWR?" H 5500 3750 50  0001 C CNN
+F 0 "#PWR0102" H 5500 3750 50  0001 C CNN
 F 1 "GND" H 5500 3850 50  0000 C CNN
 F 2 "" H 5500 4000 50  0001 C CNN
@@
 $EndComp
 $Comp
-L R_Small R102
+L Device:R_Small R2
 U 1 1 5B330CE7
 P 6050 3750
-F 0 "R102" H 6080 3770 50  0000 L CNN
+F 0 "R2" H 6080 3770 50  0000 L CNN
 F 1 "309k" H 6080 3710 50  0000 L CNN
 F 2 "Resistors_SMD:R_0603" H 6050 3750 50  0001 C CNN
@@
 $EndComp
 $Comp
-L R_Small R103
+L Device:R_Small R3
 U 1 1 5B330D2A
 P 6400 3750
-F 0 "R103" H 6430 3770 50  0000 L CNN
+F 0 "R3" H 6430 3770 50  0000 L CNN
 F 1 "1M" H 6430 3710 50  0000 L CNN
 F 2 "Resistors_SMD:R_0603" H 6400 3750 50  0001 C CNN
@@
 $EndComp
 $Comp
-L C_Small C104
+L Device:C_Small C5
 U 1 1 5B330DA5
 P 6400 3600
-F 0 "C104" H 6410 3670 50  0000 L CNN
+F 0 "C5" H 6410 3670 50  0000 L CNN
 F 1 "10pF" H 6410 3520 50  0000 L CNN
 F 2 "Capacitors_SMD:C_0603" H 6400 3600 50  0001 C CNN
@@
 $EndComp
 $Comp
-L C_Small C105
+L Device:C_Small C6
 U 1 1 5B330DFE
 P 6700 3800
-F 0 "C105" H 6710 3870 50  0000 L CNN
+F 0 "C6" H 6710 3870 50  0000 L CNN
 F 1 "22uF" H 6710 3720 50  0000 L CNN
 F 2 "Capacitors_SMD:C_0603" H 6700 3800 50  0001 C CNN
@@
 $EndComp
 Wire Wire Line
-	4550 3000 5000 3000
+	4550 3000 4700 3000
 Wire Wire Line
 	5000 3100 4900 3100
@@
 	4600 3700 4600 4000
 Wire Wire Line
-	4600 4000 6700 4000
+	4600 4000 4750 4000
 Wire Wire Line
 	5500 4000 5500 3950
@@
 Connection ~ 4750 4000
 Wire Wire Line
-	6000 3600 6300 3600
+	6000 3600 6050 3600
 Wire Wire Line
 	6050 3650 6050 3600
@@
 	6500 3600 6550 3600
 Wire Wire Line
-	6550 3600 6550 3750
+	6550 3600 6550 3650
 Wire Wire Line
 	6550 3750 6500 3750
 Wire Wire Line
-	6700 3200 6700 3700
+	6700 3200 6700 3650
 Wire Wire Line
 	6700 3650 6550 3650
@@
 Connection ~ 6700 3650
 $Comp
-L L_Small L100
+L Device:L_Small L1
 U 1 1 5B330F62
 P 6400 3200
-F 0 "L100" H 6450 3250 50  0000 L CNN
+F 0 "L1" H 6450 3250 50  0000 L CNN
 F 1 "2.2uH" H 6430 3160 50  0000 L CNN
 F 2 "Inductors_SMD:L_Vishay_IHLP-2020" H 6400 3200 50  0001 C CNN
@@
 $EndComp
 $Comp
-L C_Small C103
+L Device:C_Small C4
 U 1 1 5B330FC3
 P 6150 3000
-F 0 "C103" H 6160 3070 50  0000 L CNN
+F 0 "C4" H 6160 3070 50  0000 L CNN
 F 1 "0.1uF" H 6160 2920 50  0000 L CNN
 F 2 "Capacitors_SMD:C_0603" H 6150 3000 50  0001 C CNN
@@
 	6000 3000 6050 3000
 Wire Wire Line
-	6000 3200 6300 3200
-Wire Wire Line
-	6500 3200 6950 3200
+	6000 3200 6250 3200
+Wire Wire Line
+	6500 3200 6600 3200
 Connection ~ 6700 3200
 Wire Wire Line
@@
 Connection ~ 6250 3200
 Wire Wire Line
-	6000 3500 6950 3500
-$Comp
-L R_Small R101
+	6000 3500 6600 3500
+$Comp
+L Device:R_Small R4
 U 1 1 5B3311CE
 P 6600 3350
-F 0 "R101" H 6630 3370 50  0000 L CNN
+F 0 "R4" H 6630 3370 50  0000 L CNN
 F 1 "100k" H 6630 3310 50  0000 L CNN
 F 2 "Resistors_SMD:R_0603" H 6600 3350 50  0001 C CNN
@@
 Text HLabel 6950 3500 2    60   Input ~ 0
 P_GOOD
+Wire Wire Line
+	4900 3000 5000 3000
+Wire Wire Line
+	4700 3000 4900 3000
+Wire Wire Line
+	4900 4000 5500 4000
+Wire Wire Line
+	4750 4000 4900 4000
+Wire Wire Line
+	6050 3600 6250 3600
+Wire Wire Line
+	6250 3600 6300 3600
+Wire Wire Line
+	6550 3650 6550 3750
+Wire Wire Line
+	6700 3650 6700 3700
+Wire Wire Line
+	6700 3200 6950 3200
+Wire Wire Line
+	6250 3200 6300 3200
+Wire Wire Line
+	6600 3200 6700 3200
+Wire Wire Line
+	6600 3500 6950 3500
+Wire Wire Line
+	5500 4000 6050 4000
+Wire Wire Line
+	6050 4000 6700 4000
+$Comp
+L lt8609:LT8609 U2
+U 1 1 5BA67E7B
+P 5500 3350
+F 0 "U2" H 5500 3947 60  0000 C CNN
+F 1 "LT8609" H 5500 3841 60  0000 C CNN
+F 2 "Housings_SSOP:MSOP-10-1EP_3x3mm_Pitch0.5mm" H 5500 3800 60  0001 C CNN
+F 3 "" H 5500 3800 60  0001 C CNN
+	1    5500 3350
+	1    0    0    -1
+$EndComp
 $EndSCHEMATC

Commit message: a bunch of stuff I guess. mostly layout.
Parts:
- removed C1: 1uF, Capacitors_SMD:C_0603, symbol Device:C_Small
- removed C2: 4.7uF, Capacitors_SMD:C_0603, symbol Device:C_Small
- removed C3: 10nF, Capacitors_SMD:C_0603, symbol Device:C_Small
- removed C4: 0.1uF, Capacitors_SMD:C_0603, symbol Device:C_Small
- removed C5: 10pF, Capacitors_SMD:C_0603, symbol Device:C_Small
- removed C6: 22uF, Capacitors_SMD:C_0603, symbol Device:C_Small
- removed L1: 2.2uH, Inductors_SMD:L_Vishay_IHLP-2020, symbol Device:L_Small
- removed R1: 18.2k, Resistors_SMD:R_0603, symbol Device:R_Small
- removed R2: 309k, Resistors_SMD:R_0603, symbol Device:R_Small
- removed R3: 1M, Resistors_SMD:R_0603, symbol Device:R_Small
- removed R4: 100k, Resistors_SMD:R_0603, symbol Device:R_Small
- removed U2: LT8609, Housings_SSOP:MSOP-10-1EP_3x3mm_Pitch0.5mm, symbol lt8609:LT8609
- added C10: 47u, Capacitors_SMD:C_0603, symbol Device:C
- added C6: 2.2u, Capacitors_SMD:C_0603, symbol Device:C
- added C7: 330p, Capacitors_SMD:C_0603, symbol Device:C
- added C8: 22u, Capacitors_SMD:C_0603, symbol Device:C
- added C9: 0.1u, Capacitors_SMD:C_0603, symbol Device:C
- added L1: 1u, Inductors_SMD:L_Vishay_IHLP-1616, symbol pspice:INDUCTOR
- added R2: 20k, Resistors_SMD:R_0603, symbol Device:R
- added R3: 324k, Resistors_SMD:R_0603, symbol Device:R
- added R4: 115k, Resistors_SMD:R_0603, symbol Device:R
- added R5: 25.5, Resistors_SMD:R_0603, symbol Device:R
- added U1: LTC3604_UD, Housings_DFN_QFN:QFN-16-1EP_3x3mm_Pitch0.5mm_ThermalVias, symbol Exodus_PowerRegulator:LTC3604_UD
Connections:
- net labels added: BST, FB, INTVcc, ITH, PG, PGND, PGOOD, RT, SGND, SW, Von
- net labels removed: P_GOOD
- wire segments 47 -> 34

Commit message: updated power supply circuit. Better bandwidth, added softstart cap
Parts:
- added C1: 2200p, Capacitors_SMD:C_0603, symbol Device:C
- L1: value 1u -> 0.47u
- R3: value 324k -> 210k
Connections:
- wire segments 34 -> 37
Changed lines of the file:
@@
 F 0 "U1" H 5200 4300 50  0000 C CNN
 F 1 "LTC3604_UD" H 6100 4300 50  0000 C CNN
-F 2 "Housings_DFN_QFN:QFN-16-1EP_3x3mm_Pitch0.5mm_ThermalVias" H 5750 4500 50  0001 C CNN
+F 2 "Housings_DFN_QFN:QFN-16-1EP_3x3mm_Pitch0.5mm_ThermalVias" H 5750 4500 50  0000 C CNN
 F 3 "" H 5700 3950 50  0001 C CNN
 	1    5750 3650
@@
 P 7100 3550
 F 0 "L1" H 7100 3765 50  0000 C CNN
-F 1 "1u" H 7100 3674 50  0000 C CNN
+F 1 "0.47u" H 7100 3674 50  0000 C CNN
 F 2 "Inductors_SMD:L_Vishay_IHLP-1616" H 7100 3550 50  0001 C CNN
 F 3 "" H 7100 3550 50  0001 C CNN
@@
 P 4750 4100
 F 0 "R3" H 4820 4146 50  0000 L CNN
-F 1 "324k" H 4820 4055 50  0000 L CNN
+F 1 "210k" H 4820 4055 50  0000 L CNN
 F 2 "Resistors_SMD:R_0603" V 4680 4100 50  0001 C CNN
 F 3 "~" H 4750 4100 50  0001 C CNN
@@
 Text Label 5000 3350 0    50   ~ 0
 PG
+Wire Wire Line
+	5050 3450 3600 3450
+$Comp
+L Device:C C1
+U 1 1 5C56BE8A
+P 3600 3950
+F 0 "C1" H 3715 3996 50  0000 L CNN
+F 1 "2200p" H 3715 3905 50  0000 L CNN
+F 2 "Capacitors_SMD:C_0603" H 3638 3800 50  0001 C CNN
+F 3 "~" H 3600 3950 50  0001 C CNN
+	1    3600 3950
+	1    0    0    -1
+$EndComp
+$Comp
+L power:GND #PWR0101
+U 1 1 5C56BEBC
+P 3600 4250
+F 0 "#PWR0101" H 3600 4000 50  0001 C CNN
+F 1 "GND" H 3605 4077 50  0000 C CNN
+F 2 "" H 3600 4250 50  0001 C CNN
+F 3 "" H 3600 4250 50  0001 C CNN
+	1    3600 4250
+	1    0    0    -1
+$EndComp
+Wire Wire Line
+	3600 4250 3600 4100
+Wire Wire Line
+	3600 3450 3600 3800
 $EndSCHEMATC

Commit message: redirected 3D models for custom footprints on PCB
Parts:
- U1: footprint Housings_DFN_QFN:QFN-16-1EP_3x3mm_Pitch0.5mm_ThermalVias -> Exodus_Packages:QFN-16-1EP_3x3mm_P0.5mm
Changed lines of the file:
@@
 F 0 "U1" H 5200 4300 50  0000 C CNN
 F 1 "LTC3604_UD" H 6100 4300 50  0000 C CNN
-F 2 "Housings_DFN_QFN:QFN-16-1EP_3x3mm_Pitch0.5mm_ThermalVias" H 5750 4500 50  0000 C CNN
+F 2 "Exodus_Packages:QFN-16-1EP_3x3mm_P0.5mm" H 5750 4500 50  0000 C CNN
 F 3 "" H 5700 3950 50  0001 C CNN
 	1    5750 3650
