File: ethernet_phy_ksz8081.sch (KiCad schematic (older format))
At the start: 14 parts

Commit message: More phy progress
Parts:
- added R?: 10K, symbol Device:R
- added R?: 1K, symbol Device:R
- added R?: 10K DNP, symbol Device:R
- added R?: 1M DNP, symbol Device:R
- R?: value 10K -> 1K
Connections:
- net labels added: 1.2V_INTERNALLY_REGULATED, INTRP, OSC_OUT, REF_CLK_50MHZ, RMII_CRS_DV, RMII_MDC, RMII_MDIO, RMII_REF_CLK_OUT, RMII_RXD0, RMII_RXD1, RMII_RXER, RMII_TXD0, RMII_TXD1, RMII_TXEN, ~RST~
- net labels removed: 1.2V_PHY_INTERNALLY_REGULATED, PHY_OSC_OUT, PHY_REF_CLK_50MHZ, PHY_RMII_MDC, PHY_RMII_MDIO, PHY_RMII_REF_CLK_OUT, PHY_RMII_RXER
- wire segments 34 -> 54
Other:
- note added: "Only place if a pull-up is\nnot placed elsewhere"
- moved on the sheet: R?

Commit message: Finished PHY circuit.
Parts:
- removed TP? (x2): Test_Point, symbol Connector:Test_Point
- added TP1, TP2: TestPoint, symbol Connector:TestPoint
- C10, C11, C12, C7, C8, C9: renamed from C?; footprint (none) -> Capacitors_SMD:C_0603
- R10, R11, R5, R6, R7, R8, R9: renamed from R?; footprint (none) -> Resistors_SMD:R_0603
- U3: renamed from U?; footprint Package_DFN_QFN:QFN-24-1EP_4x4mm_P0.5mm_EP2.6x2.6mm -> Housings_DFN_QFN:QFN-20-1EP_4x4mm_Pitch0.5mm
- gave numbers to parts that had none: 2
Connections:
- net labels added: LED0, RXM, RXP, TXM, TXP
- wire segments 54 -> 55

Commit message: a bunch of stuff I guess. mostly layout.
Parts:
- R13: renamed from R12; footprint (none) -> Resistors_SMD:R_0603
- U2: renamed from U3; footprint Housings_DFN_QFN:QFN-20-1EP_4x4mm_Pitch0.5mm -> Housings_DFN_QFN:QFN-24-1EP_4x4mm_Pitch0.5mm
- renumbered C7 to C11, C8 to C12, C9 to C13, C10 to C14, C11 to C15, C12 to C16, R9 to R10, R10 to R11, R11 to R12, R5 to R6, R6 to R7, R7 to R8, R8 to R9
Changed lines of the file:
@@
 $EndDescr
 $Comp
-L Device:C C8
+L Device:C C12
 U 1 1 5B79DE1B
 P 4450 2900
-F 0 "C8" H 4565 2946 50  0000 L CNN
+F 0 "C12" H 4565 2946 50  0000 L CNN
 F 1 "22u" H 4565 2855 50  0000 L CNN
 F 2 "Capacitors_SMD:C_0603" H 4488 2750 50  0001 C CNN
@@
 $EndComp
 $Comp
-L Device:C C10
+L Device:C C14
 U 1 1 5B79DE89
 P 4900 2900
-F 0 "C10" H 5015 2946 50  0000 L CNN
+F 0 "C14" H 5015 2946 50  0000 L CNN
 F 1 "0.1u" H 5015 2855 50  0000 L CNN
 F 2 "Capacitors_SMD:C_0603" H 4938 2750 50  0001 C CNN
@@
 $EndComp
 $Comp
-L power:GND #PWR0103
+L power:GND #PWR038
 U 1 1 5B79E51C
 P 4450 3050
-F 0 "#PWR0103" H 4450 2800 50  0001 C CNN
+F 0 "#PWR038" H 4450 2800 50  0001 C CNN
 F 1 "GND" H 4455 2877 50  0000 C CNN
 F 2 "" H 4450 3050 50  0001 C CNN
@@
 $EndComp
 $Comp
-L power:GND #PWR0104
+L power:GND #PWR040
 U 1 1 5B79E535
 P 4900 3050
-F 0 "#PWR0104" H 4900 2800 50  0001 C CNN
+F 0 "#PWR040" H 4900 2800 50  0001 C CNN
 F 1 "GND" H 4905 2877 50  0000 C CNN
 F 2 "" H 4900 3050 50  0001 C CNN
@@
 $EndComp
 $Comp
-L Device:C C11
+L Device:C C15
 U 1 1 5B79EAF1
 P 6300 2100
-F 0 "C11" H 6415 2146 50  0000 L CNN
+F 0 "C15" H 6415 2146 50  0000 L CNN
 F 1 "22u" H 6415 2055 50  0000 L CNN
 F 2 "Capacitors_SMD:C_0603" H 6338 1950 50  0001 C CNN
@@
 $EndComp
 $Comp
-L Device:C C12
+L Device:C C16
 U 1 1 5B79EAF7
 P 6750 2100
-F 0 "C12" H 6865 2146 50  0000 L CNN
+F 0 "C16" H 6865 2146 50  0000 L CNN
 F 1 "0.1u" H 6865 2055 50  0000 L CNN
 F 2 "Capacitors_SMD:C_0603" H 6788 1950 50  0001 C CNN
@@
 $EndComp
 $Comp
-L power:GND #PWR0105
+L power:GND #PWR042
 U 1 1 5B79EAFD
 P 6300 2250
-F 0 "#PWR0105" H 6300 2000 50  0001 C CNN
+F 0 "#PWR042" H 6300 2000 50  0001 C CNN
 F 1 "GND" H 6305 2077 50  0000 C CNN
 F 2 "" H 6300 2250 50  0001 C CNN
@@
 $EndComp
 $Comp
-L power:GND #PWR0106
+L power:GND #PWR044
 U 1 1 5B79EB03
 P 6750 2250
-F 0 "#PWR0106" H 6750 2000 50  0001 C CNN
+F 0 "#PWR044" H 6750 2000 50  0001 C CNN
 F 1 "GND" H 6755 2077 50  0000 C CNN
 F 2 "" H 6750 2250 50  0001 C CNN
@@
 $EndComp
 $Comp
-L Device:C C7
+L Device:C C11
 U 1 1 5B79EBAF
 P 4450 2100
-F 0 "C7" H 4565 2146 50  0000 L CNN
+F 0 "C11" H 4565 2146 50  0000 L CNN
 F 1 "22u" H 4565 2055 50  0000 L CNN
 F 2 "Capacitors_SMD:C_0603" H 4488 1950 50  0001 C CNN
@@
 $EndComp
 $Comp
-L Device:C C9
+L Device:C C13
 U 1 1 5B79EBB5
 P 4900 2100
-F 0 "C9" H 5015 2146 50  0000 L CNN
+F 0 "C13" H 5015 2146 50  0000 L CNN
 F 1 "0.1u" H 5015 2055 50  0000 L CNN
 F 2 "Capacitors_SMD:C_0603" H 4938 1950 50  0001 C CNN
@@
 $EndComp
 $Comp
-L power:GND #PWR0107
+L power:GND #PWR037
 U 1 1 5B79EBBB
 P 4450 2250
-F 0 "#PWR0107" H 4450 2000 50  0001 C CNN
+F 0 "#PWR037" H 4450 2000 50  0001 C CNN
 F 1 "GND" H 4455 2077 50  0000 C CNN
 F 2 "" H 4450 2250 50  0001 C CNN
@@
 $EndComp
 $Comp
-L power:GND #PWR0108
+L power:GND #PWR039
 U 1 1 5B79EBC1
 P 4900 2250
-F 0 "#PWR0108" H 4900 2000 50  0001 C CNN
+F 0 "#PWR039" H 4900 2000 50  0001 C CNN
 F 1 "GND" H 4905 2077 50  0000 C CNN
 F 2 "" H 4900 2250 50  0001 C CNN
@@
 	5450 1750 4900 1750
 $Comp
-L power:+3.3V #PWR0109
+L power:+3.3V #PWR043
 U 1 1 5B7A0EBC
 P 6750 1650
-F 0 "#PWR0109" H 6750 1500 50  0001 C CNN
+F 0 "#PWR043" H 6750 1500 50  0001 C CNN
 F 1 "+3.3V" H 6765 1823 50  0000 C CNN
 F 2 "" H 6750 1650 50  0001 C CNN
@@
 Connection ~ 6750 1750
 $Comp
-L power:GND #PWR0110
+L power:GND #PWR041
 U 1 1 5B7A147B
 P 5850 5600
-F 0 "#PWR0110" H 5850 5350 50  0001 C CNN
+F 0 "#PWR041" H 5850 5350 50  0001 C CNN
 F 1 "GND" H 5855 5427 50  0000 C CNN
 F 2 "" H 5850 5600 50  0001 C CNN
@@
 To the layout guy: put everything up here close to the phy, numb-nuts
 $Comp
-L Device:R R12
+L Device:R R13
 U 1 1 5B7A1FD9
 P 7200 5350
-F 0 "R12" H 7270 5396 50  0000 L CNN
+F 0 "R13" H 7270 5396 50  0000 L CNN
 F 1 "6.49K 1%" H 7270 5305 50  0000 L CNN
-F 2 "" V 7130 5350 50  0001 C CNN
+F 2 "Resistors_SMD:R_0603" V 7130 5350 50  0001 C CNN
 F 3 "~" H 7200 5350 50  0001 C CNN
 	1    7200 5350
@@
 $EndComp
 $Comp
-L power:GND #PWR0111
+L power:GND #PWR045
 U 1 1 5B7A2272
 P 7200 5500
-F 0 "#PWR0111" H 7200 5250 50  0001 C CNN
+F 0 "#PWR045" H 7200 5250 50  0001 C CNN
 F 1 "GND" H 7205 5327 50  0000 C CNN
 F 2 "" H 7200 5500 50  0001 C CNN
@@
 RMII_MDC
 $Comp
-L Device:R R5
+L Device:R R6
 U 1 1 5B7A99EA
 P 1750 3300
-F 0 "R5" H 1820 3346 50  0000 L CNN
+F 0 "R6" H 1820 3346 50  0000 L CNN
 F 1 "1K" H 1820 3255 50  0000 L CNN
 F 2 "Resistors_SMD:R_0603" V 1680 3300 50  0001 C CNN
@@
 $EndComp
 $Comp
-L Device:R R6
+L Device:R R7
 U 1 1 5B7A9A2C
 P 2150 3300
-F 0 "R6" H 2220 3346 50  0000 L CNN
+F 0 "R7" H 2220 3346 50  0000 L CNN
 F 1 "1M DNP" H 2220 3255 50  0000 L CNN
 F 2 "Resistors_SMD:R_0603" V 2080 3300 50  0001 C CNN
@@
 $EndComp
 $Comp
-L power:+3.3V #PWR0112
+L power:+3.3V #PWR030
 U 1 1 5B7AAA93
 P 1750 3150
-F 0 "#PWR0112" H 1750 3000 50  0001 C CNN
+F 0 "#PWR030" H 1750 3000 50  0001 C CNN
 F 1 "+3.3V" H 1765 3323 50  0000 C CNN
 F 2 "" H 1750 3150 50  0001 C CNN
@@
 $EndComp
 $Comp
-L power:+3.3V #PWR0113
+L power:+3.3V #PWR031
 U 1 1 5B7AAAD6
 P 2150 3150
-F 0 "#PWR0113" H 2150 3000 50  0001 C CNN
+F 0 "#PWR031" H 2150 3000 50  0001 C CNN
 F 1 "+3.3V" H 2165 3323 50  0000 C CNN
 F 2 "" H 2150 3150 50  0001 C CNN
@@
 RMII_RXER
 $Comp
-L Device:R R9
+L Device:R R10
 U 1 1 5B7B046C
 P 3500 5700
-F 0 "R9" H 3570 5746 50  0000 L CNN
+F 0 "R10" H 3570 5746 50  0000 L CNN
 F 1 "1K" H 3570 5655 50  0000 L CNN
 F 2 "Resistors_SMD:R_0603" V 3430 5700 50  0001 C CNN
@@
 $EndComp
 $Comp
-L power:GND #PWR0114
+L power:GND #PWR034
 U 1 1 5B7B0E7F
 P 3500 5850
-F 0 "#PWR0114" H 3500 5600 50  0001 C CNN
+F 0 "#PWR034" H 3500 5600 50  0001 C CNN
 F 1 "GND" H 3505 5677 50  0000 C CNN
 F 2 "" H 3500 5850 50  0001 C CNN
@@
 RMII_REF_CLK_OUT
 $Comp
-L Interface_Ethernet:KSZ8081RND U3
+L Interface_Ethernet:KSZ8081RND U2
 U 1 1 5B7B87DF
 P 5850 4600
-F 0 "U3" H 5300 3550 50  0000 C CNN
+F 0 "U2" H 5300 3550 50  0000 C CNN
 F 1 "KSZ8081RND" H 5500 3650 50  0000 C CNN
-F 2 "Housings_DFN_QFN:QFN-20-1EP_4x4mm_Pitch0.5mm" H 7250 3600 50  0001 C CNN
+F 2 "Housings_DFN_QFN:QFN-24-1EP_4x4mm_Pitch0.5mm" H 7250 3600 50  0001 C CNN
 F 3 "http://ww1.microchip.com/downloads/en/DeviceDoc/00002199A.pdf" H 3600 4800 50  0001 C CNN
 	1    5850 4600
@@
 The MCU must provide\na 50MHz reference clock
 $Comp
-L Device:R R7
+L Device:R R8
 U 1 1 5B86517F
 P 2600 3300
-F 0 "R7" H 2670 3346 50  0000 L CNN
+F 0 "R8" H 2670 3346 50  0000 L CNN
 F 1 "1K" H 2670 3255 50  0000 L CNN
 F 2 "Resistors_SMD:R_0603" V 2530 3300 50  0001 C CNN
@@
 $EndComp
 $Comp
-L power:+3.3V #PWR0115
+L power:+3.3V #PWR032
 U 1 1 5B865185
 P 2600 3150
-F 0 "#PWR0115" H 2600 3000 50  0001 C CNN
+F 0 "#PWR032" H 2600 3000 50  0001 C CNN
 F 1 "+3.3V" H 2615 3323 50  0000 C CNN
 F 2 "" H 2600 3150 50  0001 C CNN
@@
 Only place if a pull-up is\nnot placed elsewhere
 $Comp
-L Device:R R8
+L Device:R R9
 U 1 1 5B86CA8D
 P 3050 3300
-F 0 "R8" H 3120 3346 50  0000 L CNN
+F 0 "R9" H 3120 3346 50  0000 L CNN
 F 1 "10K DNP" H 3120 3255 50  0000 L CNN
 F 2 "Resistors_SMD:R_0603" V 2980 3300 50  0001 C CNN
@@
 $EndComp
 $Comp
-L power:+3.3V #PWR0116
+L power:+3.3V #PWR033
 U 1 1 5B86CA93
 P 3050 3150
-F 0 "#PWR0116" H 3050 3000 50  0001 C CNN
+F 0 "#PWR033" H 3050 3000 50  0001 C CNN
 F 1 "+3.3V" H 3065 3323 50  0000 C CNN
 F 2 "" H 3050 3150 50  0001 C CNN
@@
 Connection ~ 3500 4300
 $Comp
-L Device:R R10
+L Device:R R11
 U 1 1 5B8621BD
 P 3900 5700
-F 0 "R10" H 3970 5746 50  0000 L CNN
+F 0 "R11" H 3970 5746 50  0000 L CNN
 F 1 "10K" H 3970 5655 50  0000 L CNN
 F 2 "Resistors_SMD:R_0603" V 3830 5700 50  0001 C CNN
@@
 $EndComp
 $Comp
-L power:GND #PWR0117
+L power:GND #PWR035
 U 1 1 5B862370
 P 3900 5850
-F 0 "#PWR0117" H 3900 5600 50  0001 C CNN
+F 0 "#PWR035" H 3900 5600 50  0001 C CNN
 F 1 "GND" H 3905 5677 50  0000 C CNN
 F 2 "" H 3900 5850 50  0001 C CNN
@@
 	6550 4200 8650 4200
 $Comp
-L Device:R R11
+L Device:R R12
 U 1 1 5B870A0C
 P 4250 5700
-F 0 "R11" H 4320 5746 50  0000 L CNN
+F 0 "R12" H 4320 5746 50  0000 L CNN
 F 1 "1M DNP" H 4320 5655 50  0000 L CNN
 F 2 "Resistors_SMD:R_0603" V 4180 5700 50  0001 C CNN
@@
 	4250 3700 5150 3700
 $Comp
-L power:GND #PWR0118
+L power:GND #PWR036
 U 1 1 5B8718F6
 P 4250 5850
-F 0 "#PWR0118" H 4250 5600 50  0001 C CNN
+F 0 "#PWR036" H 4250 5600 50  0001 C CNN
 F 1 "GND" H 4255 5677 50  0000 C CNN
 F 2 "" H 4250 5850 50  0001 C CNN

Commit message: layout
Parts:
- L2: footprint (none) -> Inductors_SMD:L_0603
Changed lines of the file:
@@
 F 0 "L2" V 5974 1750 50  0000 C CNN
 F 1 "Ferrite_Bead" V 5883 1750 50  0000 C CNN
-F 2 "" V 5630 1750 50  0001 C CNN
+F 2 "Inductors_SMD:L_0603" V 5630 1750 50  0001 C CNN
 F 3 "~" H 5700 1750 50  0001 C CNN
 	1    5700 1750

Commit message: revised ethernet layout
Parts:
- R10, R11, R6, R8: footprint Resistors_SMD:R_0603 -> Resistor_SMD:R_0603_1608Metric
- R12, R7, R9: footprint Resistors_SMD:R_0603 -> (none)
Changed lines of the file:
@@
 F 0 "R6" H 1820 3346 50  0000 L CNN
 F 1 "1K" H 1820 3255 50  0000 L CNN
-F 2 "Resistors_SMD:R_0603" V 1680 3300 50  0001 C CNN
+F 2 "Resistor_SMD:R_0603_1608Metric" V 1680 3300 50  0001 C CNN
 F 3 "~" H 1750 3300 50  0001 C CNN
 	1    1750 3300
@@
 F 0 "R7" H 2220 3346 50  0000 L CNN
 F 1 "1M DNP" H 2220 3255 50  0000 L CNN
-F 2 "Resistors_SMD:R_0603" V 2080 3300 50  0001 C CNN
+F 2 "" V 2080 3300 50  0001 C CNN
 F 3 "~" H 2150 3300 50  0001 C CNN
 	1    2150 3300
@@
 F 0 "R10" H 3570 5746 50  0000 L CNN
 F 1 "1K" H 3570 5655 50  0000 L CNN
-F 2 "Resistors_SMD:R_0603" V 3430 5700 50  0001 C CNN
+F 2 "Resistor_SMD:R_0603_1608Metric" V 3430 5700 50  0001 C CNN
 F 3 "~" H 3500 5700 50  0001 C CNN
 	1    3500 5700
@@
 F 0 "R8" H 2670 3346 50  0000 L CNN
 F 1 "1K" H 2670 3255 50  0000 L CNN
-F 2 "Resistors_SMD:R_0603" V 2530 3300 50  0001 C CNN
+F 2 "Resistor_SMD:R_0603_1608Metric" V 2530 3300 50  0001 C CNN
 F 3 "~" H 2600 3300 50  0001 C CNN
 	1    2600 3300
@@
 F 0 "R9" H 3120 3346 50  0000 L CNN
 F 1 "10K DNP" H 3120 3255 50  0000 L CNN
-F 2 "Resistors_SMD:R_0603" V 2980 3300 50  0001 C CNN
+F 2 "" V 2980 3300 50  0001 C CNN
 F 3 "~" H 3050 3300 50  0001 C CNN
 	1    3050 3300
@@
 F 0 "R11" H 3970 5746 50  0000 L CNN
 F 1 "10K" H 3970 5655 50  0000 L CNN
-F 2 "Resistors_SMD:R_0603" V 3830 5700 50  0001 C CNN
+F 2 "Resistor_SMD:R_0603_1608Metric" V 3830 5700 50  0001 C CNN
 F 3 "~" H 3900 5700 50  0001 C CNN
 	1    3900 5700
@@
 Text HLabel 1500 3700 0    50   Input ~ 0
 RMII_TXEN
-Wire Wire Line
-	1500 3700 4250 3700
 Text HLabel 1500 3800 0    50   Input ~ 0
 RMII_TXD0
@@
 Wire Wire Line
 	6550 4200 8650 4200
-$Comp
-L Device:R R12
-U 1 1 5B870A0C
-P 4250 5700
-F 0 "R12" H 4320 5746 50  0000 L CNN
-F 1 "1M DNP" H 4320 5655 50  0000 L CNN
-F 2 "Resistors_SMD:R_0603" V 4180 5700 50  0001 C CNN
-F 3 "~" H 4250 5700 50  0001 C CNN
-	1    4250 5700
-	1    0    0    -1
-$EndComp
-Wire Wire Line
-	4250 5550 4250 3700
-Connection ~ 4250 3700
-Wire Wire Line
-	4250 3700 5150 3700
-$Comp
-L power:GND #PWR036
-U 1 1 5B8718F6
-P 4250 5850
-F 0 "#PWR036" H 4250 5600 50  0001 C CNN
-F 1 "GND" H 4255 5677 50  0000 C CNN
-F 2 "" H 4250 5850 50  0001 C CNN
-F 3 "" H 4250 5850 50  0001 C CNN
-	1    4250 5850
-	1    0    0    -1
-$EndComp
 $Comp
 L Connector:TestPoint TP1
@@
 Text HLabel 8650 4800 2    50   Input ~ 0
 LED0
+Wire Wire Line
+	4250 3700 5150 3700
+Wire Wire Line
+	1500 3700 4250 3700
+Connection ~ 4250 3700
+Wire Wire Line
+	4250 5550 4250 3700
+$Comp
+L power:GND #PWR036
+U 1 1 5B8718F6
+P 4250 5850
+F 0 "#PWR036" H 4250 5600 50  0001 C CNN
+F 1 "GND" H 4255 5677 50  0000 C CNN
+F 2 "" H 4250 5850 50  0001 C CNN
+F 3 "" H 4250 5850 50  0001 C CNN
+	1    4250 5850
+	1    0    0    -1
+$EndComp
+$Comp
+L Device:R R12
+U 1 1 5B870A0C
+P 4250 5700
+F 0 "R12" H 4320 5746 50  0000 L CNN
+F 1 "1M DNP" H 4320 5655 50  0000 L CNN
+F 2 "" V 4180 5700 50  0001 C CNN
+F 3 "~" H 4250 5700 50  0001 C CNN
+	1    4250 5700
+	1    0    0    -1
+$EndComp
 $EndSCHEMATC
